File: flex/flex.kicad_pcb (KiCad board)
At the start: 2 copper layers, 126.3 x 113 mm, 105 parts, among them J1 Conn_01x06_Female, J2 Conn_01x05_Female, J3 Conn_01x03_Female, J4 Conn_01x06_Female, J5 Conn_01x03_Female, SW1 SW_Push, SW10 SW_Push, SW11 SW_Push, SW12 SW_Push, SW14 SW_Push, SW15 SW_Push, SW16 SW_Push, SW17 SW_Push, SW19 SW_Push, SW2 SW_Push, SW20 SW_Push, SW21 SW_Push, SW22 SW_Push, SW23 SW_Push, SW24 SW_Push, SW25 SW_Push, SW26 SW_Push, SW3 SW_Push, SW4 SW_Push, SW5 SW_Push, SW6 SW_Push, SW7 SW_Push, SW8 SW_Push, SW9 SW_Push

Commit message: WIP
Parts:
- removed C2: C, Capacitor_SMD:C_1206_3216Metric_Pad1.42x1.75mm_HandSolder
- removed D20, D22, D24, D26, D27, D28, D29, D30, D34, D36, D38, D40, D42, D44, D46, D48, D50, D52, D54, D56, D58, D6, D60, D8: SK6812MINI, libs2:YS-SK6812MINI-E_REVERSE_NO_EDGECUT
- removed the G*** at (366.7, 111.2)
- removed the G*** at (277.7, 122.3)
- removed the G*** at (278.1, 122.6)
- removed the G*** at (366.4, 111.2)
- removed the G*** at (266.9, 142.5)
- removed the G*** at (267.0, 148.6)
- D1, D10, D11, D12, D13, D14, D15, D16, D17, D31, D32, D9: value D_Schottky_x2_KCom_AAK -> D_BAV70
- SW1, SW10, SW11, SW12, SW14, SW15, SW16, SW17, SW19, SW2, SW20, SW21, SW22, SW23, SW24, SW25, SW26, SW3, SW4, SW5, SW6, SW7, SW8: footprint custom:SW_MX_reversible -> prettylib:MX100-ChocV1V2-flex; moved to F.Cu
- SW9: footprint custom:SW_MX_reversible -> prettylib:MX100-ChocV1V2-flex
- moved D57 10.2 mm to (154.2, 85.4)
- moved D19 10.1 mm to (87.2, 38.3)
- moved D53 10.1 mm to (154.2, 39.5)
- moved D59 9.96 mm to (154.2, 108.4)
- moved D41 9.95 mm to (109.2, 59.0)
- moved D33 9.87 mm to (65.2, 73.2)
- moved D47 9.86 mm to (132.7, 62.5)
- moved D55 9.81 mm to (154.2, 62.5)
- moved D7 9.80 mm to (65.2, 96.2)
- moved D45 9.80 mm to (132.7, 39.6)
- moved D4 9.78 mm to (43.7, 96.2)
- moved D3 9.72 mm to (43.7, 73.3)
- moved D51 9.71 mm to (132.7, 108.4)
- moved D21 9.71 mm to (87.3, 61.3)
- moved D43 9.71 mm to (109.2, 36.1)
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Routing:
- net Vcc: track 926.6 -> 2.66 mm, vias 28 -> 0
- net Gnd: track 897.9 -> 2.76 mm, vias 36 -> 0
- net row1: track 655.7 -> 0.00 mm, vias 6 -> 0
- net row2: track 513.7 -> 0.00 mm, vias 13 -> 0
- net row4: track 431.2 -> 0.00 mm, vias 7 -> 0
- net col1: track 286.0 -> 0.00 mm, vias 5 -> 0
- net col2: track 273.8 -> 0.00 mm, vias 8 -> 0
- net row3: track 262.8 -> 0.00 mm, vias 3 -> 0
- net col3: track 218.7 -> 0.00 mm, vias 5 -> 0
- net col6: track 204.1 -> 0.00 mm, vias 6 -> 0
- net Net-(D43-DOUT): track 192.7 -> 0.00 mm, vias 3 -> 0
- net Net-(D19-DIN): track 164.0 -> 0.00 mm, vias 4 -> 0
- net col5: track 160.7 -> 0.00 mm, vias 3 -> 0
- net col4: track 131.7 -> 0.00 mm, vias 5 -> 0
- net Net-(D51-DOUT): track 126.2 -> 0.00 mm, vias 4 -> 0
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- removed copper zone on B.Cu, net Gnd
- removed copper zone on F.Cu, net Gnd
Other:
- board text removed: "Conn_01x06_Female"
- board text removed: "Conn_01x07_Female"
- board text removed: "D"
- board text removed: "J1"
- board text removed: "J10"
- board text removed: "J11"
- board text removed: "J12"
- board text removed: "J13"
- board text removed: "J14"
- board text removed: "J15"
- board text removed: "J2"
- board text removed: "J3"
- board text removed: "J4"
- board text removed: "J5"
- board text removed: "J6"
- board text removed: "J7"
- board text removed: "J8"
- board text removed: "J9"
- board text removed: "SW1"
- board text removed: "SW10"
- board text removed: "SW11"
- board text removed: "SW12"
- board text removed: "SW13"
- board text removed: "SW14"
- board text removed: "SW15"
- board text removed: "SW16"
- board text removed: "SW17"
- board text removed: "SW18"
- board text removed: "SW19"
- board text removed: "SW2"
- board text removed: "SW20"
- board text removed: "SW21"
- board text removed: "SW22"
- board text removed: "SW23"
- board text removed: "SW24"
- board text removed: "SW25"
- board text removed: "SW26"
- board text removed: "SW27"
- board text removed: "SW28"
- board text removed: "SW29"
- board text removed: "SW3"
- board text removed: "SW30"
- board text removed: "SW31"
- board text removed: "SW32"
- board text removed: "SW4"
- board text removed: "SW5"
- board text removed: "SW6"
- board text removed: "SW7"
- board text removed: "SW8"
- board text removed: "SW9"
- board text removed: "SW_Push"
