File: flex/flex.kicad_sch (KiCad schematic)
At the start: 93 parts, among them J1 Conn_01x06_Female, J2 Conn_01x05_Female, J3 Conn_01x03_Female, J4 Conn_01x06_Female, J5 Conn_01x03_Female, SW1 SW_Push, SW10 SW_Push, SW11 SW_Push, SW12 SW_Push, SW14 SW_Push, SW15 SW_Push, SW16 SW_Push, SW17 SW_Push, SW19 SW_Push, SW2 SW_Push, SW20 SW_Push, SW21 SW_Push, SW22 SW_Push, SW23 SW_Push, SW24 SW_Push, SW25 SW_Push, SW26 SW_Push, SW3 SW_Push, SW4 SW_Push, SW5 SW_Push, SW6 SW_Push, SW7 SW_Push, SW8 SW_Push, SW9 SW_Push

Commit message: WIP
Parts:
- removed C2: C, Capacitor_SMD:C_1206_3216Metric_Pad1.42x1.75mm_HandSolder, symbol Device:C
- removed D20, D22, D24, D26, D27, D28, D29, D30, D34, D36, D38, D40, D42, D44, D46, D48, D50, D52, D54, D56, D58, D6, D60, D8: SK6812MINI, libs2:YS-SK6812MINI-E_REVERSE_NO_EDGECUT, symbol LED:SK6812MINI
- D1, D10, D11, D12, D13, D14, D15, D16, D17, D31, D32, D9: value D_Schottky_x2_KCom_AAK -> D_BAV70; symbol Device:D_Schottky_x2_KCom_AAK -> kbd:D_BAV70; LCSC (none) -> C68978
- SW1, SW10, SW11, SW12, SW14, SW15, SW16, SW17, SW19, SW2, SW20, SW21, SW22, SW23, SW24, SW25, SW26, SW3, SW4, SW5, SW6, SW7, SW8, SW9: footprint custom:SW_MX_reversible -> prettylib:MX100-ChocV1V2-flex
