File: flex/flex.kicad_sch (KiCad schematic)
At the start: 93 parts, among them J1 Conn_01x06_Female, J2 Conn_01x05_Female, J3 Conn_01x03_Female, J4 Conn_01x06_Female, J5 Conn_01x03_Female, SW1 SW_Push, SW10 SW_Push, SW11 SW_Push, SW12 SW_Push, SW14 SW_Push, SW15 SW_Push, SW16 SW_Push, SW17 SW_Push, SW19 SW_Push, SW2 SW_Push, SW20 SW_Push, SW21 SW_Push, SW22 SW_Push, SW23 SW_Push, SW24 SW_Push, SW25 SW_Push, SW26 SW_Push, SW3 SW_Push, SW4 SW_Push, SW5 SW_Push, SW6 SW_Push, SW7 SW_Push, SW8 SW_Push, SW9 SW_Push

Commit message: new
Parts:
- removed D20, D22, D24, D26, D27, D28, D29, D30, D34, D36, D38, D40, D42, D44, D46, D48, D50, D52, D54, D56, D58, D6, D60, D8: SK6812MINI, libs2:YS-SK6812MINI-E_REVERSE_NO_EDGECUT, symbol LED:SK6812MINI
- removed R1, R2: R, Resistor_SMD:R_1206_3216Metric_Pad1.42x1.75mm_HandSolder, symbol Device:R
- added C3, C4, C5, C6: C, Capacitor_SMD:C_0805_2012Metric, symbol Device:C
- C1, C2: footprint Capacitor_SMD:C_1206_3216Metric_Pad1.42x1.75mm_HandSolder -> Capacitor_SMD:C_0805_2012Metric
- D1, D10, D11, D12, D13, D14, D15, D16, D17, D31, D32, D9: value D_Schottky_x2_KCom_AAK -> D_BAV70; footprint customs:TSOT-23_HandSoldering -> prettylib:TSOT-23_HandSoldering; symbol Device:D_Schottky_x2_KCom_AAK -> kbd:D_BAV70; LCSC (none) -> C68978
- D18, D19, D2, D21, D23, D25, D3, D33, D35, D37, D39, D4, D41, D43, D45, D47, D49, D5, D51, D53, D55, D57, D59, D7: footprint libs2:YS-SK6812MINI-E_REVERSE -> prettylib:YS-SK6812MINI-E-bkb; symbol LED:SK6812MINI -> kbd:SK6803MINI-E
- SW1, SW10, SW11, SW12, SW14, SW15, SW16, SW17, SW19, SW2, SW20, SW21, SW22, SW23, SW24, SW25, SW26, SW3, SW4, SW5, SW6, SW7, SW8, SW9: footprint custom:SW_MX_reversible -> prettylib:SW_MX_KS_Choc-mod; symbol Switch:SW_Push -> kbd:SW_Push
Connections:
- net Din: now also D2.3 (DIN)
- net Gnd: now also C3.2, C4.2, C5.2, C6.2
- net Vcc: now also C3.1, C4.1, C5.1, C6.1
- net row1: now also SW1.2, SW14.2, SW19.2, SW23.2, SW5.2, SW9.2; no longer SW1.1, SW14.1, SW19.1, SW23.1, SW5.1, SW9.1
- net row2: now also SW10.2, SW15.2, SW2.2, SW20.2, SW24.2, SW6.2; no longer SW10.1, SW15.1, SW2.1, SW20.1, SW24.1, SW6.1
- net row3: now also SW11.2, SW16.2, SW21.2, SW25.2, SW3.2, SW7.2; no longer SW11.1, SW16.1, SW21.1, SW25.1, SW3.1, SW7.1
- net row4: now also SW12.2, SW17.2, SW22.2, SW26.2, SW4.2, SW8.2; no longer SW12.1, SW17.1, SW22.1, SW26.1, SW4.1, SW8.1
- net at D15.1 (A): now also SW22.1; no longer SW22.2
- net at D15.2 (A): now also SW21.1; no longer SW21.2
- net at D13.1 (A): now also SW2.1; no longer SW2.2
- net at D17.1 (A): now also SW26.1; no longer SW26.2
- net at D17.2 (A): now also SW25.1; no longer SW25.2
- net at D31.2 (A): now also SW5.1; no longer SW5.2
- net at D10.2 (A): now also SW11.1; no longer SW11.2
- net at D10.1 (A): now also SW12.1; no longer SW12.2
- net at D32.1 (A): now also SW8.1; no longer SW8.2
- net at D12.1 (A): now also SW17.1; no longer SW17.2
- net at D12.2 (A): now also SW16.1; no longer SW16.2
- net at D31.1 (A): now also SW6.1; no longer SW6.2
- net at D13.2 (A): now also SW1.1; no longer SW1.2
- net at D1.2 (A): now also SW3.1; no longer SW3.2
- net at D11.2 (A): now also SW14.1; no longer SW14.2
- net at D16.1 (A): now also SW24.1; no longer SW24.2
- net at D9.1 (A): now also SW10.1; no longer SW10.2
- net at D9.2 (A): now also SW9.1; no longer SW9.2
- net at D14.1 (A): now also SW20.1; no longer SW20.2
- net at D11.1 (A): now also SW15.1; no longer SW15.2
- net at D1.1 (A): now also SW4.1; no longer SW4.2
- net at D14.2 (A): now also SW19.1; no longer SW19.2
- net at D32.2 (A): now also SW7.1; no longer SW7.2
- net at D16.2 (A): now also SW23.1; no longer SW23.2
Other:
- note added: "Reversed"
